Commit message: Finish two-robot launch file and workspace

File: urdf/workspace.urdf.xacro (robot description, xacro)
@@ -3,4 +3,21 @@
   <!-- Pull in the UR macro (contains UR3/5/10/16 including e-series) -->
   <xacro:include filename="$(find ur_description)/urdf/ur_macro.xacro"/>
+  <!-- Fro control tag -->
+  <xacro:include filename="$(find ur_description)/urdf/ur.ros2_control.xacro"/>
+  <!-- parameters -->
+  <xacro:arg name="joint_limit_params" default="$(find ur_description)/config/ur5e/joint_limits.yaml"/>
+  <xacro:arg name="kinematics_params" default="$(find ur_description)/config/ur5e/default_kinematics.yaml"/>
+  <xacro:arg name="physical_params" default="$(find ur_description)/config/ur5e/physical_parameters.yaml"/>
+  <xacro:arg name="visual_params" default="$(find ur_description)/config/ur5e/visual_parameters.yaml"/>
+  <xacro:arg name="ur_script_filename" default="$(find ur_client_library)/resources/external_control.urscript"/>
+  <xacro:arg name="ur_output_recipe_filename" default="$(find ur_robot_driver)/resources/rtde_output_recipe.txt"/>
+  <xacro:arg name="ur_input_recipe_filename" default="$(find ur_robot_driver)/resources/rtde_input_recipe.txt"/>
+  <!-- initial position for simulations (Fake Hardware, Gazebo, Ignition) -->
+  <xacro:arg name="initial_positions_file" default="$(find ur_description)/config/initial_positions.yaml"/>
+  <xacro:arg name="script_filename" default="$(find ur_client_library)/resources/external_control.urscript"/>
+  <xacro:arg name="input_recipe_filename" default="$(find ur_robot_driver)/resources/rtde_input_recipe.txt"/>
+  <xacro:arg name="output_recipe_filename" default="$(find ur_robot_driver)/resources/rtde_output_recipe.txt"/>
+  <!-- convert to property to use substitution in function -->
+  <xacro:property name="initial_positions_file" default="$(arg initial_positions_file)"/>
   <!-- Root -->
   <link name="world">
@@ -26,11 +43,4 @@
   </joint>
   <!-- Robots -->
-  <!-- import main macro -->
-  <xacro:include filename="$(find ur_description)/urdf/ur_macro.xacro"/>
-  <!-- parameters -->
-  <xacro:arg name="joint_limit_params" default="$(find ur_description)/config/ur5e/joint_limits.yaml"/>
-  <xacro:arg name="kinematics_params" default="$(find ur_description)/config/ur5e/default_kinematics.yaml"/>
-  <xacro:arg name="physical_params" default="$(find ur_description)/config/ur5e/physical_parameters.yaml"/>
-  <xacro:arg name="visual_params" default="$(find ur_description)/config/ur5e/visual_parameters.yaml"/>
   <xacro:ur_robot
       name="left_ur5e"
@@ -41,6 +51,15 @@
       physical_parameters_file="$(arg physical_params)"
       visual_parameters_file="$(arg visual_params)"
-      robot_ip="10.164.8.235">
-    <origin xyz="0.5 -0.2 0" rpy="0 0 0" />
+      initial_positions="${xacro.load_yaml(initial_positions_file)}"
+      robot_ip="10.164.8.235"
+      reverse_ip="0.0.0.0"
+      script_filename="$(arg script_filename)"
+      output_recipe_filename="$(arg output_recipe_filename)"
+      input_recipe_filename="$(arg input_recipe_filename)"
+      script_command_port="50004"
+      reverse_port="50001"
+      script_sender_port="50002"
+      trajectory_port="50003">
+    <origin xyz="0.25 -0.4 0" rpy="0 0 1.5708" />
   </xacro:ur_robot>
   <xacro:ur_robot
@@ -52,6 +71,15 @@
       physical_parameters_file="$(arg physical_params)"
       visual_parameters_file="$(arg visual_params)"
-      robot_ip="10.164.8.222">
-    <origin xyz="-0.5 -0.2 0" rpy="0 0 0" />
+      initial_positions="${xacro.load_yaml(initial_positions_file)}"
+      robot_ip="10.164.8.222"
+      reverse_ip="0.0.0.0"
+      script_filename="$(arg script_filename)"
+      output_recipe_filename="$(arg output_recipe_filename)"
+      input_recipe_filename="$(arg input_recipe_filename)"
+      script_command_port="50008"
+      reverse_port="50005"
+      script_sender_port="50006"
+      trajectory_port="50007">
+    <origin xyz="-0.25 -0.4 0" rpy="0 0 1.5708" />
   </xacro:ur_robot>
 </robot>

Commit message: Working two robot driver and jerky GoC-MPC node

File: urdf/workspace.urdf.xacro (robot description, xacro)
@@ -61,5 +61,5 @@
       script_sender_port="50002"
       trajectory_port="50003">
-    <origin xyz="0.25 -0.4 0" rpy="0 0 1.5708" />
+    <origin xyz="0.3 -0.4 0" rpy="0 0 1.5708" />
   </xacro:ur_robot>
   <xacro:ur_robot
@@ -81,5 +81,5 @@
       script_sender_port="50006"
       trajectory_port="50007">
-    <origin xyz="-0.25 -0.4 0" rpy="0 0 1.5708" />
+    <origin xyz="-0.3 -0.4 0" rpy="0 0 1.5708" />
   </xacro:ur_robot>
 </robot>

Commit message: Tweaks for frames and get twist from robot

File: urdf/workspace.urdf.xacro (robot description, xacro)
@@ -53,5 +53,5 @@
       initial_positions="${xacro.load_yaml(initial_positions_file)}"
       robot_ip="10.164.8.235"
-      reverse_ip="0.0.0.0"
+      reverse_ip="10.164.8.247"
       script_filename="$(arg script_filename)"
       output_recipe_filename="$(arg output_recipe_filename)"
@@ -61,5 +61,5 @@
       script_sender_port="50002"
       trajectory_port="50003">
-    <origin xyz="0.3 -0.4 0" rpy="0 0 1.5708" />
+    <origin xyz="0.36 -0.7 0" rpy="0 0 1.5708" />
   </xacro:ur_robot>
   <xacro:ur_robot
@@ -73,5 +73,5 @@
       initial_positions="${xacro.load_yaml(initial_positions_file)}"
       robot_ip="10.164.8.222"
-      reverse_ip="0.0.0.0"
+      reverse_ip="10.164.8.247"
       script_filename="$(arg script_filename)"
       output_recipe_filename="$(arg output_recipe_filename)"
@@ -81,5 +81,5 @@
       script_sender_port="50006"
       trajectory_port="50007">
-    <origin xyz="-0.3 -0.4 0" rpy="0 0 1.5708" />
+    <origin xyz="-0.36 -0.7 0" rpy="0 0 1.5708" />
   </xacro:ur_robot>
 </robot>

Commit message: Camera alignment stuff and gripper support. Almost complete

File: urdf/workspace.urdf.xacro (robot description, xacro)
@@ -40,5 +40,5 @@
     <parent link="world"/>
     <child link="camera_link"/>
-    <origin xyz="0.0 1.0 0.20" rpy="0 0 -1.5708"/>
+    <origin xyz="0.0 1.25 0.20" rpy="0 0 -1.5708"/>
   </joint>
   <!-- Robots -->
